File: PCB_Design/PCB_Design.kicad_pcb (KiCad board)
At the start: 2 copper layers, 94.2 x 94.5 mm, 18 parts, among them U1 ESP32-DEVKITC-32E, U2 module_mpu6050, U3 YAAJ_DCDC_StepDown_LM2596, U4 ZC323200

Commit message: Auther: Ziad, Breif: add videos
Parts:
- renumbered TMC1 to TMC2209, TMC2 to TMC2209
Changed lines of the file:
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@@
 		(layer "F.Cu")
 		(at 124.7 117.1 180)
-		(property "Reference" "TMC1"
-			(at -6.3 12.2 0)
+		(property "Reference" "TMC2209"
+			(at 1.675 9.05 0)
 			(unlocked yes)
 			(layer "F.SilkS")
@@
 		(layer "F.Cu")
 		(at 148.3 117.5 180)
-		(property "Reference" "TMC2"
-			(at -6.675 12.125 0)
-			(unlocked yes)
-			(layer "F.SilkS")
+		(property "Reference" "TMC2209"
+			(at -7.9 9.65 0)
+			(unlocked yes)
+			(layer "F.SilkS")
